Commit message: fix(urdf): add missing material color definitions
Add yellow, magenta, cyan, orange, purple, pink, and brown materials
to match the color palette used in gym_bridge_launch.py. This fixes
undefined material warnings for racecars beyond the first 3.

File: src/f1tenth_gym_ros/launch/ego_racecar.xacro (robot description, xacro)
@@ -24,4 +24,25 @@
   <material name="green">
     <color rgba="0.0 1.0 0.0 1."/>
+  </material>
+  <material name="yellow">
+    <color rgba="1.0 1.0 0.0 1."/>
+  </material>
+  <material name="magenta">
+    <color rgba="1.0 0.0 1.0 1."/>
+  </material>
+  <material name="cyan">
+    <color rgba="0.0 1.0 1.0 1."/>
+  </material>
+  <material name="orange">
+    <color rgba="1.0 0.5 0.0 1."/>
+  </material>
+  <material name="purple">
+    <color rgba="0.5 0.0 0.5 1."/>
+  </material>
+  <material name="pink">
+    <color rgba="1.0 0.75 0.8 1."/>
+  </material>
+  <material name="brown">
+    <color rgba="0.6 0.3 0.0 1."/>
   </material>
   <link name="$(arg car)/base_link">
